Commit message: Completed

File: ws3/src/metafly_description/urdf/metafly_macro.xacro (robot description, xacro)
@@ -2,14 +2,12 @@
 <robot xmlns:xacro="http://wiki.ros.org/xacro">
   <xacro:macro name="metafly" params="prefix">
-  <xacro:property name="body_length" value="0.25" />
-  <xacro:property name="body_radius" value="0.025" />
-  <xacro:property name="wing_thickness" value="0.001" />
-  <xacro:property name="wing_length" value="${body_length}" />
-  <xacro:property name="wing_width" value="0.25" />
-  <xacro:property name="wing_thickness" value="0.001" />
-    <!-- LINKS -->
-    <!-- base link -->
+    <!-- Make everything larger and easier to see -->
+    <xacro:property name="body_length" value="0.6" />
+    <xacro:property name="body_radius" value="0.06" />
+    <xacro:property name="wing_length" value="0.5" />
+    <xacro:property name="wing_width" value="0.25" />
+    <xacro:property name="wing_thickness" value="0.05" />
+    <!-- Base/body -->
     <link name="${prefix}base_link">
-      <!-- body -->
       <visual>
         <origin xyz="0 0 0" rpy="${radians(90)} 0 0" />
@@ -19,34 +17,33 @@
         <material name="light_grey"/>
       </visual>
-      <!-- head -->
       <visual>
         <origin xyz="0 ${body_length/2} 0" rpy="0 0 0" />
         <geometry>
-          <sphere radius="${body_radius*1.5}"/>
+          <sphere radius="0.09"/>
         </geometry>
+        <material name="blue"/>
       </visual>
     </link>
-    <!-- wing 1 -->
+    <!-- Left wing -->
     <link name="${prefix}wing1">
       <visual>
-        <origin xyz="${-wing_width/2} 0 0" rpy="0 0 0" />
+        <origin xyz="-0.35 0 0" rpy="0 0 0" />
         <geometry>
-          <box size="${wing_width} ${wing_length} ${wing_thickness}" />
+          <box size="0.7 0.2 0.05" />
         </geometry>
         <material name="red"/>
       </visual>
     </link>
-  <!-- wing 2 -->
+    <!-- Right wing -->
     <link name="${prefix}wing2">
       <visual>
-        <origin xyz="${wing_width/2} 0 0" rpy="0 0 0" />
+        <origin xyz="0.35 0 0" rpy="0 0 0" />
         <geometry>
-          <box size="${wing_width} ${wing_length} ${wing_thickness}" />
+          <box size="0.7 0.2 0.05" />
         </geometry>
         <material name="green"/>
       </visual>
     </link>
-    <!-- JOINTS -->
-    <!-- joint 1 -->
+    <!-- Joints -->
     <joint name="${prefix}joint1" type="revolute">
       <origin xyz="0 0 0" rpy="0 0 0" />
@@ -54,7 +51,6 @@
       <child link="${prefix}wing1" />
       <axis xyz="0 1 0" />
-      <limit effort="0" lower="${radians(-90)}" upper="${radians(90)}" velocity="0" />
+      <limit effort="1" lower="${radians(-90)}" upper="${radians(90)}" velocity="1" />
     </joint>
-    <!-- joint 2 -->
     <joint name="${prefix}joint2" type="revolute">
       <origin xyz="0 0 0" rpy="0 0 0" />
@@ -62,7 +58,6 @@
       <child link="${prefix}wing2" />
       <axis xyz="0 1 0" />
-      <limit effort="0" lower="${radians(-90)}" upper="${radians(90)}" velocity="0" />
+      <limit effort="1" lower="${radians(-90)}" upper="${radians(90)}" velocity="1" />
     </joint>
-    <!-- END JOINTS -->
   </xacro:macro>
 </robot>
